File: design/immo_board/Driver/driver.sch (EAGLE design)
At the start: 41 parts, among them IC1 7812TV, IC10 7805TV, IC2 LM393N, IC3 74LS241N, IC4 7812TV, IC5 7812TV, IC6 7812TV, IC7 7812TV, IC8 7805TV, IC9 7805TV

Commit message: Fix driver scheme (supply switch)
Parts:
- removed PAD2, PAD4: WIREPAD4,16O1,6, wirepad:WIREPAD4,16O1,6
- added BATTERY+, SWITCH_PIN1: WIREPAD4,16O1,6, wirepad:WIREPAD4,16O1,6
- renumbered PAD1 to SWITCH_PIN2, PAD3 to BATTERY-
Connections:
- net VCC: now also BATTERY+.P, SWITCH_PIN1.P; no longer PAD2.P, PAD4.P
Changed lines of the file:
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@@
 <part name="P+14" library="supply1" deviceset="+5V" device=""/>
 <part name="P+15" library="supply1" deviceset="+5V" device=""/>
-<part name="PAD1" library="wirepad" deviceset="WIREPAD" device="4,16O1,6"/>
-<part name="PAD2" library="wirepad" deviceset="WIREPAD" device="4,16O1,6"/>
+<part name="SWITCH_PIN2" library="wirepad" deviceset="WIREPAD" device="4,16O1,6"/>
+<part name="BATTERY+" library="wirepad" deviceset="WIREPAD" device="4,16O1,6"/>
 <part name="GND11" library="supply1" deviceset="GND" device=""/>
 <part name="P+3" library="supply1" deviceset="VCC" device=""/>
-<part name="PAD3" library="wirepad" deviceset="WIREPAD" device="4,16O1,6"/>
-<part name="PAD4" library="wirepad" deviceset="WIREPAD" device="4,16O1,6"/>
+<part name="BATTERY-" library="wirepad" deviceset="WIREPAD" device="4,16O1,6"/>
+<part name="SWITCH_PIN1" library="wirepad" deviceset="WIREPAD" device="4,16O1,6"/>
 <part name="P+16" library="supply1" deviceset="+18V" device=""/>
 <part name="GND13" library="supply1" deviceset="GND" device=""/>
@@
 <part name="C5" library="resistor" deviceset="CPOL-EU" device="E5-8.5"/>
 <part name="C6" library="resistor" deviceset="CPOL-EU" device="E2.5-5"/>
+<part name="SWITCH" library="switch-omron" deviceset="D-TS" device=""/>
 </parts>
 <sheets>
@@
 </plain>
 <instances>
-<instance part="PAD1" gate="G$1" x="40.64" y="17.78"/>
-<instance part="PAD2" gate="G$1" x="40.64" y="7.62" rot="R180"/>
-<instance part="P+3" gate="VCC" x="12.7" y="22.86"/>
-<instance part="PAD3" gate="G$1" x="40.64" y="-12.7"/>
-<instance part="PAD4" gate="G$1" x="40.64" y="-2.54" rot="R180"/>
+<instance part="SWITCH_PIN2" gate="G$1" x="40.64" y="17.78"/>
+<instance part="BATTERY+" gate="G$1" x="30.48" y="-12.7" rot="R180"/>
+<instance part="P+3" gate="VCC" x="5.08" y="30.48"/>
+<instance part="BATTERY-" gate="G$1" x="40.64" y="-12.7"/>
+<instance part="SWITCH_PIN1" gate="G$1" x="30.48" y="17.78" rot="R180"/>
 <instance part="P+17" gate="1" x="60.96" y="30.48"/>
 <instance part="GND14" gate="1" x="60.96" y="-20.32"/>
 <instance part="C5" gate="G$1" x="55.88" y="5.08"/>
-<instance part="C6" gate="G$1" x="60.96" y="5.08"/>
+<instance part="C6" gate="G$1" x="66.04" y="5.08"/>
+<instance part="SWITCH" gate="G$1" x="35.56" y="17.78" rot="R270"/>
 </instances>
 <busses>
@@
 <pinref part="GND14" gate="1" pin="GND"/>
 <wire x1="60.96" y1="-12.7" x2="60.96" y2="-17.78" width="0.1524" layer="91"/>
-<pinref part="PAD3" gate="G$1" pin="P"/>
+<pinref part="BATTERY-" gate="G$1" pin="P"/>
 <wire x1="43.18" y1="-12.7" x2="60.96" y2="-12.7" width="0.1524" layer="91"/>
 <pinref part="C6" gate="G$1" pin="-"/>
-<wire x1="60.96" y1="-12.7" x2="60.96" y2="0" width="0.1524" layer="91"/>
 <junction x="60.96" y="-12.7"/>
 <pinref part="C5" gate="G$1" pin="-"/>
+<wire x1="66.04" y1="0" x2="60.96" y2="0" width="0.1524" layer="91"/>
 <wire x1="60.96" y1="0" x2="55.88" y2="0" width="0.1524" layer="91"/>
+<wire x1="60.96" y1="0" x2="60.96" y2="-12.7" width="0.1524" layer="91"/>
 <junction x="60.96" y="0"/>
 </segment>
@@
 <net name="+18V" class="0">
 <segment>
-<pinref part="PAD1" gate="G$1" pin="P"/>
+<pinref part="SWITCH_PIN2" gate="G$1" pin="P"/>
 <pinref part="P+17" gate="1" pin="+18V"/>
 <wire x1="43.18" y1="17.78" x2="60.96" y2="17.78" width="0.1524" layer="91"/>
@@
 <pinref part="C6" gate="G$1" pin="+"/>
 <wire x1="55.88" y1="7.62" x2="60.96" y2="7.62" width="0.1524" layer="91"/>
-<wire x1="60.96" y1="7.62" x2="60.96" y2="17.78" width="0.1524" layer="91"/>
+<wire x1="60.96" y1="7.62" x2="66.04" y2="7.62" width="0.1524" layer="91"/>
+<junction x="60.96" y="17.78"/>
+<wire x1="60.96" y1="17.78" x2="60.96" y2="7.62" width="0.1524" layer="91"/>
 <junction x="60.96" y="7.62"/>
-<junction x="60.96" y="17.78"/>
 </segment>
 </net>
@@
 <segment>
 <pinref part="P+3" gate="VCC" pin="VCC"/>
-<wire x1="12.7" y1="20.32" x2="12.7" y2="7.62" width="0.1524" layer="91"/>
-<pinref part="PAD2" gate="G$1" pin="P"/>
-<wire x1="12.7" y1="7.62" x2="38.1" y2="7.62" width="0.1524" layer="91"/>
-<wire x1="12.7" y1="-2.54" x2="12.7" y2="7.62" width="0.1524" layer="91"/>
-<junction x="12.7" y="7.62"/>
-<pinref part="PAD4" gate="G$1" pin="P"/>
-<wire x1="38.1" y1="-2.54" x2="12.7" y2="-2.54" width="0.1524" layer="91"/>
-</segment>
-</net>
+<wire x1="5.08" y1="27.94" x2="5.08" y2="17.78" width="0.1524" layer="91"/>
+<pinref part="BATTERY+" gate="G$1" pin="P"/>
+<wire x1="5.08" y1="-12.7" x2="5.08" y2="17.78" width="0.1524" layer="91"/>
+<junction x="5.08" y="17.78"/>
+<pinref part="SWITCH_PIN1" gate="G$1" pin="P"/>
+<wire x1="27.94" y1="17.78" x2="5.08" y2="17.78" width="0.1524" layer="91"/>
+<wire x1="27.94" y1="-12.7" x2="5.08" y2="-12.7" width="0.1524" layer="91"/>
+</segment>
+</net>
